File: design/flatmcu.kicad_pcb (KiCad board)
At the start: 4 copper layers, 77.8 x 63.2 mm, 127 parts, among them J1 Hall, J10 VBUS, J11 GND, J2 USB_B_Micro, J3 Throttle, J4 Motor_Phase_A, J5 Motor_Phase_B, J6 Motor_Phase_C, J7 SW Debug, J8 UART to HBD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

Commit message: updated for kicad 7
Other:
- net class Default removed
